Commit message: 移植过来

File: config/simulation/SO101/so101_new_calib.urdf (robot description, URDF)
Before this commit: robot so101_new_calib, 8 links, 7 joints
Links:
- link base_link: geometry collision mesh filename=assets/base_so101_v2.stl; collision mesh filename=assets/sts3215_03a_v1.stl

Commit message: 移植过来

File: config/simulation/SO101/so101_new_calib.urdf (robot description, URDF)
Before this commit: robot so101_new_calib, 8 links, 7 joints
Links:
- link base_link: geometry collision mesh filename=./config/simulation/SO101/assets/base_motor_holder_so101_v1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; collision mesh filename=assets/base_so101_v2.stl

Commit message: 移植过来

File: config/simulation/SO101/so101_new_calib.urdf (robot description, URDF)
Before this commit: robot so101_new_calib, 8 links, 7 joints
Links:
- link base_link: geometry collision mesh filename=./assets/base_motor_holder_so101_v1.stl; collision mesh filename=assets/base_so101_v2.stl
